Commit message: Switch to inmoov_urdf-master head model (25 Texture STLs)
- Replace inmoov_description meshes with the 25 head STLs from
  inmoov_urdf-master/archive/meshes/stl/ (Texture011-015, 068-087)
- Rewrite head.urdf with exact joints/origins from InMoov.urdf:
  rothead (±0.524 rad), jaw (0-0.175 rad), eye pan (±0.349 rad),
  eye tilt (±0.785 rad)
- Fix robot-viewer.js: handle multiple <visual> elements per link
  (rothead has 16, jaw has 3) using querySelectorAll instead of
  querySelector; apply MODEL_SCALE=0.1196 on root group
- Update updateRobotModel() joint names to match new URDF:
  i01.head.rothead_link_joint, i01.head.jaw_link_joint,
  i01.head.eyeLeft/Right.001_link_joint, eyeLeft/Right_link_joint

Co-Authored-By: Claude Sonnet 4.6 <noreply@anthropic.com>

File: public/robot/head.urdf (robot description, URDF)
Before this commit: robot inmoov_head, 17 links, 16 joints
Links:
- removed link eyesupport_link
- removed link face_link
- removed link head_base_link
- removed link head_link
- removed link jaw_link
- removed link l_camera_link
- removed link l_eye_link
- removed link l_eyesupport_link
- removed link l_iris_link
- removed link left_ear_link
- removed link r_camera_link
- removed link r_eye_link
- removed link r_eyesupport_link
- removed link r_iris_link
- removed link right_ear_link
- removed link skull_link
- added link i01.head.eyeLeft.001_link
- added link i01.head.eyeLeft_link; visual mesh filename=/robot/meshes/Texture011.stl scale=1 1 1
- added link i01.head.eyeRight.001_link
- added link i01.head.eyeRight_link; visual mesh filename=/robot/meshes/Texture012.stl scale=1 1 1
- added link i01.head.jaw_link; visual mesh filename=/robot/meshes/Texture014.stl scale=1 1 1; visual mesh filename=/robot/meshes/Texture086.stl scale=1 1 1
- added link i01.head.rothead_link; visual mesh filename=/robot/meshes/Texture013.stl scale=1 1 1; visual mesh filename=/robot/meshes/Texture068.stl scale=1 1 1
- added link neck_link; visual mesh filename=/robot/meshes/Texture015.stl scale=1 1 1; visual mesh filename=/robot/meshes/Texture083.stl scale=1 1 1
Joints:
- removed joint base_to_base
- removed joint eyes_pan_joint
- removed joint eyes_tilt_joint
- removed joint face_joint
- removed joint head_pan_joint
- removed joint jaw_joint
- removed joint l_camera_joint
- removed joint l_eye_joint
- removed joint l_eye_pan_joint
- removed joint l_iris_joint
- removed joint left_ear_joint
- removed joint r_camera_joint
- removed joint r_eye_joint
- removed joint r_iris_joint
- removed joint right_ear_joint
- removed joint skull_joint
- added joint base_to_neck: type fixed, parent base_link, child neck_link, origin xyz=0 0 0 rpy=0 0 0
- added joint i01.head.eyeLeft.001_link_joint: type revolute, parent i01.head.rothead_link, child i01.head.eyeLeft.001_link, origin xyz=-1.08601 -0.29198 0.37576 rpy=0 0 -1.57080, axis 0 0 1, limit lower=-0.34907 upper=0.34907 effort=0 velocity=0.78540
- added joint i01.head.eyeLeft_link_joint: type revolute, parent i01.head.eyeLeft.001_link, child i01.head.eyeLeft_link, origin xyz=0 -0.00590 0 rpy=0 0 0, axis 0.99994 0 0.01111, limit lower=-0.78530 upper=0.78530 effort=0 velocity=0.78540
- added joint i01.head.eyeRight.001_link_joint: type revolute, parent i01.head.rothead_link, child i01.head.eyeRight.001_link, origin xyz=-1.09644 0.29850 0.37576 rpy=0 0 -1.57080, axis 0 0 1, limit lower=-0.34907 upper=0.34907 effort=0 velocity=0.78540
- added joint i01.head.eyeRight_link_joint: type revolute, parent i01.head.eyeRight.001_link, child i01.head.eyeRight_link, origin xyz=0 -0.00590 0 rpy=0 0 0, axis 0.99994 0 0.01111, limit lower=-0.78530 upper=0.78530 effort=0 velocity=0.78540
- added joint i01.head.jaw_link_joint: type revolute, parent i01.head.rothead_link, child i01.head.jaw_link, origin xyz=-0.36176 0.01121 0.32442 rpy=0 0 -1.57080, axis 0.99994 0 0.01111, limit lower=0 upper=0.17453 effort=0 velocity=0.78540
- added joint i01.head.rothead_link_joint: type revolute, parent neck_link, child i01.head.rothead_link, origin xyz=0.00246 0.01503 0.24911 rpy=0 0 1.57080, axis 0 0 1, limit lower=-0.52360 upper=0.52360 effort=0 velocity=0.78540

Commit message: feat(videocall): TalkBack accessibility pass, speaker mute, theme setting, 0-90 head range
Accessibility (blind operator is a primary user):
- Fix aria-pressed on every toggle to the same convention: pressed=true
  means the feature is ON (mic/camera/speaker were inverted).
- Replace scattered aria-live regions with two dedicated sr-status nodes
  (polite + assertive) driven by announceAccessibility(); drop aria-live
  from room code, MQTT status and chat so TalkBack stops interrupting.
- Add sr-only eye D-pad buttons and expose the eye stick as an ARIA
  slider, so eye control is reachable without pointer gestures.
- Tap-boost the head/mouth D-pad and announce resulting angles.
- Mark decorative nodes (login bg/logo, avatar, cam placeholder,
  joystick thumb) aria-hidden; login error gets role="alert".
- Thai-only button labels and titles.

Controls and media:
- New speaker toggle that gates all TTS output.
- Joystick haptics on step boundaries.
- Whisper fallback when browser speech recognition is unavailable.
- Light/dark theme setting applied via data-theme before first paint.

Robot wire format:
- Head range 0-90 (center 45) instead of 0-80 (center 40); mouth mapping
  normalised to 30-100 across app.js, face/index.html and the docs.
- Widen the URDF rothead joint limit to +/-45 degrees to match.
- face/index.html now uses the same-origin /ws/mqtt proxy instead of
  test.mosquitto.org, so it follows localhost or the tunnel URL.

Co-Authored-By: Claude Opus 5 <noreply@anthropic.com>

File: public/robot/head.urdf (robot description, URDF)
Before this commit: robot inmoov_head, 8 links, 7 joints
Joints:
- joint i01.head.rothead_link_joint: limit lower=-0.52360 upper=0.52360 effort=0 velocity=0.78540 -> lower=-0.78540 upper=0.78540 effort=0 velocity=0.78540
